File: SolarFlowmeterMonitor/SolarFlowmeterMonitor.kicad_pcb (KiCad board)
At the start: 2 copper layers, 18 parts, among them J1 FlowMeter, J2 SP-pins, J3 Conn_01x10_Pin, J4 Solar Panel 280mA@18V, Q1 AO3413, Q2 2N7000, U1 StepDown_LM2596, U2 XL6009, U3 LoadSharing, U4 LiCharger, U7 XC6206P332MR

Commit message: fixes
Parts:
- moved U2 79.5 mm to (144.7, 101.5), turned to -90 degrees
- moved U4 34.1 mm to (130.5, 76.6), turned to 90 degrees
- moved U3 18.6 mm to (123.7, 105.9)
- moved U1 16.4 mm to (70.2, 111.0)
Connections:
- J3 pad 2: BAT+ -> GND
- U3 pad 2: BAT+ -> +5VSP
- U4 pad 1: (no net) -> +5VSP
- U4 pad 2: (no net) -> GND
Routing:
- net GND: vias 8 -> 9
Other:
- board text added: "SFM uSPX@2026"
